Commit message: Modification of the center wheel

File: ros2_ws/src/mobile_robot_description/urdf/mobile_robot.urdf.xacro (robot description, xacro)
@@ -3,6 +3,8 @@
     <xacro:property name="block_width" value="0.2"/>
     <xacro:property name="block_height" value="0.2"/>
-    <xacro:property name="wheel_radius" value="0.08"/>
-    <xacro:property name="wheel_width" value="0.04"/>
+    <xacro:property name="main_wheel_radius" value="0.08"/>
+    <xacro:property name="main_wheel_width" value="0.04"/>
+    <xacro:property name="center_wheel_radius" value="0.04"/>
+    <xacro:property name="center_wheel_width" value="0.02"/>
     <link name="base_link">
       <visual>
@@ -17,5 +19,5 @@
       </collision>
     </link>
-    <xacro:macro name="wheel" params="name parent x y z">
+    <xacro:macro name="wheel" params="name parent x y z wheel_radius wheel_width">
       <link name="${name}_wheel_link">
         <visual>
@@ -39,5 +41,6 @@
       </joint>
     </xacro:macro>
-    <xacro:wheel name="left" parent="base_link" x="0" y="${block_width/2 + wheel_width/2}" z="-${block_height/4}"/>
-    <xacro:wheel name="right" parent="base_link" x="0" y="${-block_width/2 - wheel_width/2}" z="-${block_height/4}"/>
+    <xacro:wheel name="left" parent="base_link" x="${block_length/4}" y="${block_width/2 + main_wheel_width/2}" z="-${block_height/4}" wheel_radius="${main_wheel_radius}" wheel_width="${main_wheel_width}"/>
+    <xacro:wheel name="right" parent="base_link" x="${block_length/4}" y="${-block_width/2 - main_wheel_width/2}" z="-${block_height/4}" wheel_radius="${main_wheel_radius}" wheel_width="${main_wheel_width}"/>
+    <xacro:wheel name="center" parent="base_link" x="-${block_length/4}" y="0" z="-${block_height/2}" wheel_radius="${center_wheel_radius}" wheel_width="${center_wheel_width}"/>
 </robot>

Commit message: Addition of the base_footprint for ground reference

File: ros2_ws/src/mobile_robot_description/urdf/mobile_robot.urdf.xacro (robot description, xacro)
@@ -7,4 +7,5 @@
     <xacro:property name="center_wheel_radius" value="0.04"/>
     <xacro:property name="center_wheel_width" value="0.02"/>
+    <link name="base_footprint"/>
     <link name="base_link">
       <visual>
@@ -41,6 +42,11 @@
       </joint>
     </xacro:macro>
-    <xacro:wheel name="left" parent="base_link" x="${block_length/4}" y="${block_width/2 + main_wheel_width/2}" z="-${block_height/4}" wheel_radius="${main_wheel_radius}" wheel_width="${main_wheel_width}"/>
-    <xacro:wheel name="right" parent="base_link" x="${block_length/4}" y="${-block_width/2 - main_wheel_width/2}" z="-${block_height/4}" wheel_radius="${main_wheel_radius}" wheel_width="${main_wheel_width}"/>
+    <joint name="base_footprint_joint" type="fixed">
+      <parent link="base_footprint"/>
+      <child link="base_link"/>
+      <origin xyz="0 0 ${block_height/2 + center_wheel_radius}" rpy="0 0 0"/>
+    </joint>
+    <xacro:wheel name="left" parent="base_link" x="${block_length/4}" y="${block_width/2 + main_wheel_width/2}" z="${-block_height/2 + (main_wheel_radius-center_wheel_radius)}" wheel_radius="${main_wheel_radius}" wheel_width="${main_wheel_width}"/>
+    <xacro:wheel name="right" parent="base_link" x="${block_length/4}" y="${-block_width/2 - main_wheel_width/2}" z="${-block_height/2 + (main_wheel_radius-center_wheel_radius)}" wheel_radius="${main_wheel_radius}" wheel_width="${main_wheel_width}"/>
     <xacro:wheel name="center" parent="base_link" x="-${block_length/4}" y="0" z="-${block_height/2}" wheel_radius="${center_wheel_radius}" wheel_width="${center_wheel_width}"/>
 </robot>

Commit message: Spawn Robot in Gazebo world, control with teleoperation

File: ros2_ws/src/mobile_robot_description/urdf/mobile_robot.urdf.xacro (robot description, xacro)
@@ -7,6 +7,35 @@
     <xacro:property name="center_wheel_radius" value="0.04"/>
     <xacro:property name="center_wheel_width" value="0.02"/>
+    <xacro:property name="ground_clearance" value="${center_wheel_radius}"/>
+    <xacro:property name="base_mass" value="4.0"/>
+    <xacro:property name="main_wheel_mass" value="0.3"/>
+    <xacro:property name="center_wheel_mass" value="0.1"/>
+    <xacro:macro name="box_inertia" params="mass x y z">
+      <inertial>
+        <mass value="${mass}"/>
+        <inertia
+          ixx="${mass * (y*y + z*z) / 12.0}"
+          ixy="0.0"
+          ixz="0.0"
+          iyy="${mass * (x*x + z*z) / 12.0}"
+          iyz="0.0"
+          izz="${mass * (x*x + y*y) / 12.0}"/>
+      </inertial>
+    </xacro:macro>
+    <xacro:macro name="wheel_inertia" params="mass radius width">
+      <inertial>
+        <mass value="${mass}"/>
+        <inertia
+          ixx="${mass * (3.0*radius*radius + width*width) / 12.0}"
+          ixy="0.0"
+          ixz="0.0"
+          iyy="${mass * radius*radius / 2.0}"
+          iyz="0.0"
+          izz="${mass * (3.0*radius*radius + width*width) / 12.0}"/>
+      </inertial>
+    </xacro:macro>
     <link name="base_footprint"/>
     <link name="base_link">
+      <xacro:box_inertia mass="${base_mass}" x="${block_length}" y="${block_width}" z="${block_height}"/>
       <visual>
         <geometry>
@@ -20,6 +49,7 @@
       </collision>
     </link>
-    <xacro:macro name="wheel" params="name parent x y z wheel_radius wheel_width">
+    <xacro:macro name="wheel" params="name parent x y z wheel_radius wheel_width wheel_mass">
       <link name="${name}_wheel_link">
+        <xacro:wheel_inertia mass="${wheel_mass}" radius="${wheel_radius}" width="${wheel_width}"/>
         <visual>
           <origin rpy="1.5708 0 0"/>
@@ -45,8 +75,41 @@
       <parent link="base_footprint"/>
       <child link="base_link"/>
-      <origin xyz="0 0 ${block_height/2 + center_wheel_radius}" rpy="0 0 0"/>
+      <origin xyz="0 0 ${block_height/2 + ground_clearance}" rpy="0 0 0"/>
     </joint>
-    <xacro:wheel name="left" parent="base_link" x="${block_length/4}" y="${block_width/2 + main_wheel_width/2}" z="${-block_height/2 + (main_wheel_radius-center_wheel_radius)}" wheel_radius="${main_wheel_radius}" wheel_width="${main_wheel_width}"/>
-    <xacro:wheel name="right" parent="base_link" x="${block_length/4}" y="${-block_width/2 - main_wheel_width/2}" z="${-block_height/2 + (main_wheel_radius-center_wheel_radius)}" wheel_radius="${main_wheel_radius}" wheel_width="${main_wheel_width}"/>
-    <xacro:wheel name="center" parent="base_link" x="-${block_length/4}" y="0" z="-${block_height/2}" wheel_radius="${center_wheel_radius}" wheel_width="${center_wheel_width}"/>
+    <xacro:wheel name="left" parent="base_link" x="-${block_length/4}" y="${block_width/2 + main_wheel_width/2}" z="${main_wheel_radius - block_height/2 - ground_clearance}" wheel_radius="${main_wheel_radius}" wheel_width="${main_wheel_width}" wheel_mass="${main_wheel_mass}"/>
+    <xacro:wheel name="right" parent="base_link" x="-${block_length/4}" y="${-block_width/2 - main_wheel_width/2}" z="${main_wheel_radius - block_height/2 - ground_clearance}" wheel_radius="${main_wheel_radius}" wheel_width="${main_wheel_width}" wheel_mass="${main_wheel_mass}"/>
+    <xacro:wheel name="center" parent="base_link" x="${block_length/4}" y="0" z="${center_wheel_radius - block_height/2 - ground_clearance}" wheel_radius="${center_wheel_radius}" wheel_width="${center_wheel_width}" wheel_mass="${center_wheel_mass}"/>
+    <gazebo reference="base_link">
+      <material>Gazebo/Blue</material>
+    </gazebo>
+    <gazebo reference="left_wheel_link">
+      <material>Gazebo/Black</material>
+      <mu1>1.0</mu1>
+      <mu2>1.0</mu2>
+    </gazebo>
+    <gazebo reference="right_wheel_link">
+      <material>Gazebo/Black</material>
+      <mu1>1.0</mu1>
+      <mu2>1.0</mu2>
+    </gazebo>
+    <gazebo reference="center_wheel_link">
+      <material>Gazebo/Grey</material>
+      <mu1>0.2</mu1>
+      <mu2>0.2</mu2>
+    </gazebo>
+    <gazebo>
+      <plugin
+        filename="gz-sim-diff-drive-system"
+        name="gz::sim::systems::DiffDrive">
+        <left_joint>left_wheel_joint</left_joint>
+        <right_joint>right_wheel_joint</right_joint>
+        <wheel_separation>0.24</wheel_separation>
+        <wheel_radius>${main_wheel_radius}</wheel_radius>
+        <odom_publish_frequency>30</odom_publish_frequency>
+        <max_linear_velocity>0.5</max_linear_velocity>
+        <min_linear_velocity>-0.5</min_linear_velocity>
+        <max_angular_velocity>1.5</max_angular_velocity>
+        <min_angular_velocity>-1.5</min_angular_velocity>
+      </plugin>
+    </gazebo>
 </robot>

Commit message: SLAM and restructure of the robot creation

File: ros2_ws/src/mobile_robot_description/urdf/mobile_robot.urdf.xacro (robot description, xacro)
@@ -23,5 +23,5 @@
       </inertial>
     </xacro:macro>
-    <xacro:macro name="wheel_inertia" params="mass radius width">
+    <xacro:macro name="cylinder_inertia" params="mass radius width">
       <inertial>
         <mass value="${mass}"/>
@@ -35,4 +35,10 @@
       </inertial>
     </xacro:macro>
+    <xacro:macro name="sphere_inertia" params="mass radius">
+      <inertial>
+        <mass value="${mass}"/>
+        <inertia ixx="${(2/5) * mass * (radius*radius)}" ixy="0.0" ixz="0.0" iyy="${(2/5) * mass * (radius*radius)}" iyz="0.0" izz="${(2/5) * mass * (radius*radius)}"/>
+      </inertial>
+    </xacro:macro>
     <link name="base_footprint"/>
     <link name="base_link">
@@ -49,7 +55,40 @@
       </collision>
     </link>
+    <link name="lidar_link">
+      <visual>
+        <origin rpy="0 0 0"/>
+        <geometry>
+          <cylinder radius="0.04" length="0.04"/>
+        </geometry>
+        <material name="red">
+          <color rgba="1 0 0 1"/>
+        </material>
+      </visual>
+    </link>
+    <link name="camera_link">
+      <visual>
+        <geometry>
+          <box size="0.04 0.04 0.03"/>
+        </geometry>
+        <material name="green">
+          <color rgba="0 1 0 1"/>
+        </material>
+      </visual>
+    </link>
+    <link name="imu_link"/>
+    <link name="front_caster">
+      <xacro:sphere_inertia mass="${base_mass}" radius="${center_wheel_radius}"/>
+      <visual>
+        <geometry>
+          <sphere radius="${center_wheel_radius}"/>
+        </geometry>
+        <material name="Cyan">
+          <color rgba="0 1.0 1.0 1.0"/>
+        </material>
+      </visual>
+    </link>
     <xacro:macro name="wheel" params="name parent x y z wheel_radius wheel_width wheel_mass">
       <link name="${name}_wheel_link">
-        <xacro:wheel_inertia mass="${wheel_mass}" radius="${wheel_radius}" width="${wheel_width}"/>
+        <xacro:cylinder_inertia mass="${wheel_mass}" radius="${wheel_radius}" width="${wheel_width}"/>
         <visual>
           <origin rpy="1.5708 0 0"/>
@@ -77,7 +116,26 @@
       <origin xyz="0 0 ${block_height/2 + ground_clearance}" rpy="0 0 0"/>
     </joint>
+    <joint name="lidar_joint" type="fixed">
+      <parent link="base_link"/>
+      <child link="lidar_link"/>
+      <origin xyz="${block_length/2 - 0.04} 0 ${block_height/2 + 0.02}" rpy="0 0 0"/>
+    </joint>
+    <joint name="camera_joint" type="fixed">
+      <parent link="base_link"/>
+      <child link="camera_link"/>
+      <origin xyz="${block_length/2 + 0.02} 0 0" rpy="0 0 0"/>
+    </joint>
+    <joint name="imu_joint" type="fixed">
+      <parent link="base_link"/>
+      <child link="imu_link"/>
+      <origin xyz="0 0 0.08" rpy="0 0 0"/>
+    </joint>
     <xacro:wheel name="left" parent="base_link" x="-${block_length/4}" y="${block_width/2 + main_wheel_width/2}" z="${main_wheel_radius - block_height/2 - ground_clearance}" wheel_radius="${main_wheel_radius}" wheel_width="${main_wheel_width}" wheel_mass="${main_wheel_mass}"/>
     <xacro:wheel name="right" parent="base_link" x="-${block_length/4}" y="${-block_width/2 - main_wheel_width/2}" z="${main_wheel_radius - block_height/2 - ground_clearance}" wheel_radius="${main_wheel_radius}" wheel_width="${main_wheel_width}" wheel_mass="${main_wheel_mass}"/>
-    <xacro:wheel name="center" parent="base_link" x="${block_length/4}" y="0" z="${center_wheel_radius - block_height/2 - ground_clearance}" wheel_radius="${center_wheel_radius}" wheel_width="${center_wheel_width}" wheel_mass="${center_wheel_mass}"/>
+    <joint name="caster_joint" type="fixed">
+      <parent link="base_link"/>
+      <child link="front_caster"/>
+      <origin xyz="${block_length/4} 0.0 ${center_wheel_radius - block_height/2 - ground_clearance}" rpy="0 0 0"/>
+    </joint>
     <gazebo reference="base_link">
       <material>Gazebo/Blue</material>
@@ -93,8 +151,58 @@
       <mu2>1.0</mu2>
     </gazebo>
-    <gazebo reference="center_wheel_link">
+    <gazebo reference="front_caster">
       <material>Gazebo/Grey</material>
-      <mu1>0.2</mu1>
-      <mu2>0.2</mu2>
+      <mu1>0.02</mu1>
+      <mu2>0.02</mu2>
+    </gazebo>
+    <gazebo reference="lidar_link">
+      <sensor name="lidar" type="gpu_lidar">
+        <topic>/scan</topic>
+        <update_rate>10</update_rate>
+        <ray>
+          <scan>
+            <horizontal>
+              <samples>360</samples>
+              <resolution>1</resolution>
+              <min_angle>-3.14159</min_angle>
+              <max_angle>3.14159</max_angle>
+            </horizontal>
+          </scan>
+          <range>
+            <min>0.12</min>
+            <max>8.0</max>
+            <resolution>0.01</resolution>
+          </range>
+        </ray>
+        <always_on>true</always_on>
+        <visualize>true</visualize>
+      </sensor>
+    </gazebo>
+    <gazebo reference="camera_link">
+      <sensor name="camera" type="camera">
+        <topic>/camera/image_raw</topic>
+        <update_rate>30</update_rate>
+        <camera>
+          <horizontal_fov>1.047</horizontal_fov>
+          <image>
+            <width>640</width>
+            <height>480</height>
+            <format>R8G8B8</format>
+          </image>
+          <clip>
+            <near>0.05</near>
+            <far>20.0</far>
+          </clip>
+        </camera>
+        <always_on>true</always_on>
+        <visualize>true</visualize>
+      </sensor>
+    </gazebo>
+    <gazebo reference="imu_link">
+      <sensor name="imu" type="imu">
+        <topic>/imu</topic>
+        <update_rate>100</update_rate>
+        <always_on>true</always_on>
+      </sensor>
     </gazebo>
     <gazebo>

Commit message: Logic of SLAM with EKF Lidar and Odometry + Starting of Nav2 with costmap

File: ros2_ws/src/mobile_robot_description/urdf/mobile_robot.urdf.xacro (robot description, xacro)
@@ -78,5 +78,5 @@
     <link name="imu_link"/>
     <link name="front_caster">
-      <xacro:sphere_inertia mass="${base_mass}" radius="${center_wheel_radius}"/>
+      <xacro:sphere_inertia mass="${center_wheel_mass}" radius="${center_wheel_radius}"/>
       <visual>
         <geometry>
@@ -87,4 +87,9 @@
         </material>
       </visual>
+      <collision name="front_caster_collision">
+        <geometry>
+          <sphere radius="${center_wheel_radius}"/>
+        </geometry>
+      </collision>
     </link>
     <xacro:macro name="wheel" params="name parent x y z wheel_radius wheel_width wheel_mass">
@@ -153,10 +158,11 @@
     <gazebo reference="front_caster">
       <material>Gazebo/Grey</material>
-      <mu1>0.02</mu1>
-      <mu2>0.02</mu2>
+      <mu1>0.001</mu1>
+      <mu2>0.001</mu2>
     </gazebo>
     <gazebo reference="lidar_link">
       <sensor name="lidar" type="gpu_lidar">
         <topic>/scan</topic>
+        <gz_frame_id>lidar_link</gz_frame_id>
         <update_rate>10</update_rate>
         <ray>
@@ -219,5 +225,15 @@
         <max_angular_velocity>1.5</max_angular_velocity>
         <min_angular_velocity>-1.5</min_angular_velocity>
+        <frame_id>odom</frame_id>
+        <child_frame_id>base_footprint</child_frame_id>
       </plugin>
+      <plugin
+        filename="gz-sim-joint-state-publisher-system"
+        name="gz::sim::systems::JointStatePublisher">
+        <joint_name>left_wheel_joint</joint_name>
+        <joint_name>right_wheel_joint</joint_name>
+        <topic>/joint_states</topic>
+        <update_rate>30</update_rate>
+      </plugin>
     </gazebo>
 </robot>

Commit message: Navigation through different map, reaching the yellow ball with navigation_camera. Problem with Nav2 aborting goals

File: ros2_ws/src/mobile_robot_description/urdf/mobile_robot.urdf.xacro (robot description, xacro)
@@ -76,4 +76,14 @@
       </visual>
     </link>
+    <link name="depth_camera_link">
+      <visual>
+        <geometry>
+          <box size="0.04 0.04 0.03"/>
+        </geometry>
+        <material name="purple">
+          <color rgba="0.5 0 1 1"/>
+        </material>
+      </visual>
+    </link>
     <link name="imu_link"/>
     <link name="front_caster">
@@ -131,4 +141,9 @@
       <origin xyz="${block_length/2 + 0.02} 0 0" rpy="0 0 0"/>
     </joint>
+    <joint name="depth_camera_joint" type="fixed">
+      <parent link="base_link"/>
+      <child link="depth_camera_link"/>
+      <origin xyz="${block_length/2 + 0.02} 0 0" rpy="0 0 0"/>
+    </joint>
     <joint name="imu_joint" type="fixed">
       <parent link="base_link"/>
@@ -188,4 +203,5 @@
       <sensor name="camera" type="camera">
         <topic>/camera/image_raw</topic>
+        <gz_frame_id>camera_link</gz_frame_id>
         <update_rate>30</update_rate>
         <camera>
@@ -199,4 +215,25 @@
             <near>0.05</near>
             <far>20.0</far>
+          </clip>
+        </camera>
+        <always_on>true</always_on>
+        <visualize>true</visualize>
+      </sensor>
+    </gazebo>
+    <gazebo reference="depth_camera_link">
+      <sensor name="depth_camera" type="depth_camera">
+        <topic>/camera/depth/image_raw</topic>
+        <gz_frame_id>depth_camera_link</gz_frame_id>
+        <update_rate>30</update_rate>
+        <camera>
+          <horizontal_fov>1.047</horizontal_fov>
+          <image>
+            <width>640</width>
+            <height>480</height>
+            <format>R_FLOAT32</format>
+          </image>
+          <clip>
+            <near>0.05</near>
+            <far>8.0</far>
           </clip>
         </camera>
